File: main_board.brd (EAGLE design)
At the start: 100 x 80 mm, 4 parts

Commit message: lsm330 skonczony
Parts:
- renumbered AKC+GYRO to ACC+GYRO
Connections:
- new net INT_ACC: ACC+GYRO.P20
- new net INT_GYRO: ACC+GYRO.P18
- net GND: now also ACC+GYRO.P16
Changed lines of the file:
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@@
 </autorouter>
 <elements>
-<element name="AKC+GYRO" library="sensors-akc_zyr" package="LGA_4X5X1P1_28L" value="LSM330DLC" x="15.24" y="69.85"/>
+<element name="ACC+GYRO" library="sensors-akc_zyr" package="LGA_4X5X1P1_28L" value="LSM330DLC" x="15.24" y="69.85"/>
 <element name="C1" library="resistor" package="C0805" value="" x="2.54" y="-3.81"/>
 <element name="C2" library="resistor" package="C0805" value="" x="2.54" y="-7.62"/>
@@
 <signals>
 <signal name="N$1">
-<contactref element="AKC+GYRO" pad="P15"/>
+<contactref element="ACC+GYRO" pad="P15"/>
 <contactref element="C2" pad="1"/>
 <wire x1="1.69" y1="-7.62" x2="17.5025" y2="68.6" width="0" layer="19" extent="1-1"/>
 </signal>
 <signal name="GND">
-<contactref element="AKC+GYRO" pad="P1"/>
-<contactref element="AKC+GYRO" pad="P5"/>
-<contactref element="AKC+GYRO" pad="P6"/>
-<contactref element="AKC+GYRO" pad="P2"/>
-<contactref element="AKC+GYRO" pad="P3"/>
-<contactref element="AKC+GYRO" pad="P4"/>
+<contactref element="ACC+GYRO" pad="P1"/>
+<contactref element="ACC+GYRO" pad="P5"/>
+<contactref element="ACC+GYRO" pad="P6"/>
+<contactref element="ACC+GYRO" pad="P2"/>
+<contactref element="ACC+GYRO" pad="P3"/>
+<contactref element="ACC+GYRO" pad="P4"/>
 <contactref element="C2" pad="2"/>
 <contactref element="C3" pad="-"/>
 <contactref element="C1" pad="1"/>
-<contactref element="AKC+GYRO" pad="P27"/>
-<contactref element="AKC+GYRO" pad="P26"/>
+<contactref element="ACC+GYRO" pad="P27"/>
+<contactref element="ACC+GYRO" pad="P26"/>
+<contactref element="ACC+GYRO" pad="P16"/>
 <wire x1="14.49" y1="71.6125" x2="13.99" y2="71.6125" width="0" layer="19" extent="1-1"/>
 <wire x1="12.9775" y1="71.1" x2="13.99" y2="71.6125" width="0" layer="19" extent="1-1"/>
@@
 <wire x1="12.9775" y1="69.1" x2="12.9775" y2="69.6" width="0" layer="19" extent="1-1"/>
 <wire x1="12.9775" y1="68.6" x2="12.9775" y2="69.1" width="0" layer="19" extent="1-1"/>
+<wire x1="17.5025" y1="69.1" x2="14.49" y2="71.6125" width="0" layer="19" extent="1-1"/>
 <wire x1="1.69" y1="-3.81" x2="12.9775" y2="68.6" width="0" layer="19" extent="1-1"/>
 <wire x1="3.39" y1="-7.62" x2="1.69" y2="-3.81" width="0" layer="19" extent="1-1"/>
@@
 </signal>
 <signal name="3.3V">
-<contactref element="AKC+GYRO" pad="P13"/>
-<contactref element="AKC+GYRO" pad="P12"/>
-<contactref element="AKC+GYRO" pad="P11"/>
-<contactref element="AKC+GYRO" pad="P10"/>
-<contactref element="AKC+GYRO" pad="P9"/>
-<contactref element="AKC+GYRO" pad="P7"/>
-<contactref element="AKC+GYRO" pad="P14"/>
-<contactref element="AKC+GYRO" pad="P8"/>
-<contactref element="AKC+GYRO" pad="P21"/>
-<contactref element="AKC+GYRO" pad="P25"/>
+<contactref element="ACC+GYRO" pad="P13"/>
+<contactref element="ACC+GYRO" pad="P12"/>
+<contactref element="ACC+GYRO" pad="P11"/>
+<contactref element="ACC+GYRO" pad="P10"/>
+<contactref element="ACC+GYRO" pad="P9"/>
+<contactref element="ACC+GYRO" pad="P7"/>
+<contactref element="ACC+GYRO" pad="P14"/>
+<contactref element="ACC+GYRO" pad="P8"/>
+<contactref element="ACC+GYRO" pad="P21"/>
+<contactref element="ACC+GYRO" pad="P25"/>
 <contactref element="C1" pad="2"/>
 <contactref element="C3" pad="+"/>
-<contactref element="AKC+GYRO" pad="P23"/>
-<contactref element="AKC+GYRO" pad="P22"/>
+<contactref element="ACC+GYRO" pad="P23"/>
+<contactref element="ACC+GYRO" pad="P22"/>
 <wire x1="16.49" y1="71.6125" x2="16.99" y2="71.6125" width="0" layer="19" extent="1-1"/>
 <wire x1="15.99" y1="71.6125" x2="16.49" y2="71.6125" width="0" layer="19" extent="1-1"/>
@@
 </signal>
 <signal name="SCL">
-<contactref element="AKC+GYRO" pad="P24"/>
+<contactref element="ACC+GYRO" pad="P24"/>
 </signal>
 <signal name="SDA">
-<contactref element="AKC+GYRO" pad="P28"/>
+<contactref element="ACC+GYRO" pad="P28"/>
+</signal>
+<signal name="INT_ACC">
+<contactref element="ACC+GYRO" pad="P20"/>
+</signal>
+<signal name="INT_GYRO">
+<contactref element="ACC+GYRO" pad="P18"/>
 </signal>
 </signals>
