File: main_board.sch (EAGLE design)
At the start: 4 parts

Commit message: lsm330 skonczony
Parts:
- renumbered AKC+GYRO to ACC+GYRO
Connections:
- new net INT_ACC: ACC+GYRO.INT1_A
- new net INT_GYRO: ACC+GYRO.INT1_G
- net GND: now also ACC+GYRO.DEN_G
Changed lines of the file:
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@@
 </classes>
 <parts>
-<part name="AKC+GYRO" library="sensors-akc_zyr" deviceset="LSM330DLC" device=""/>
+<part name="ACC+GYRO" library="sensors-akc_zyr" deviceset="LSM330DLC" device=""/>
 <part name="C1" library="resistor" deviceset="C-EU" device="C0805"/>
 <part name="C2" library="resistor" deviceset="C-EU" device="C0805"/>
@@
 <part name="SUPPLY2" library="SparkFun-Aesthetics" deviceset="3.3V" device=""/>
 <part name="GND3" library="supply1" deviceset="GND" device=""/>
+<part name="GND4" library="supply1" deviceset="GND" device=""/>
 </parts>
 <sheets>
@@
 </plain>
 <instances>
-<instance part="AKC+GYRO" gate="G$1" x="43.18" y="116.84"/>
+<instance part="ACC+GYRO" gate="G$1" x="43.18" y="116.84"/>
 <instance part="C1" gate="G$1" x="22.86" y="127" rot="R180"/>
 <instance part="C2" gate="G$1" x="33.02" y="142.24" rot="R270"/>
@@
 <instance part="SUPPLY2" gate="G$1" x="20.32" y="177.8"/>
 <instance part="GND3" gate="1" x="22.86" y="160.02"/>
+<instance part="GND4" gate="1" x="91.44" y="160.02"/>
 </instances>
 <busses>
@@
 <net name="N$1" class="0">
 <segment>
-<pinref part="AKC+GYRO" gate="G$1" pin="CAP"/>
+<pinref part="ACC+GYRO" gate="G$1" pin="CAP"/>
 <pinref part="C2" gate="G$1" pin="1"/>
 <wire x1="35.56" y1="142.24" x2="38.1" y2="142.24" width="0.1524" layer="91"/>
@@
 <net name="GND" class="0">
 <segment>
-<pinref part="AKC+GYRO" gate="G$1" pin="VSS"/>
+<pinref part="ACC+GYRO" gate="G$1" pin="VSS"/>
 <pinref part="GND2" gate="1" pin="GND"/>
 <pinref part="C3" gate="G$1" pin="-"/>
@@
 </segment>
 <segment>
-<pinref part="AKC+GYRO" gate="G$1" pin="SDO_A"/>
-<pinref part="AKC+GYRO" gate="G$1" pin="SDO_G"/>
+<pinref part="ACC+GYRO" gate="G$1" pin="SDO_A"/>
+<pinref part="ACC+GYRO" gate="G$1" pin="SDO_G"/>
 <wire x1="38.1" y1="157.48" x2="38.1" y2="162.56" width="0.1524" layer="91"/>
 <wire x1="38.1" y1="162.56" x2="22.86" y2="162.56" width="0.1524" layer="91"/>
@@
 <junction x="38.1" y="162.56"/>
 </segment>
+<segment>
+<pinref part="ACC+GYRO" gate="G$1" pin="DEN_G"/>
+<pinref part="GND4" gate="1" pin="GND"/>
+<wire x1="81.28" y1="162.56" x2="91.44" y2="162.56" width="0.1524" layer="91"/>
+</segment>
 </net>
 <net name="3.3V" class="0">
 <segment>
-<pinref part="AKC+GYRO" gate="G$1" pin="VDD"/>
-<pinref part="AKC+GYRO" gate="G$1" pin="VDD_IO"/>
+<pinref part="ACC+GYRO" gate="G$1" pin="VDD"/>
+<pinref part="ACC+GYRO" gate="G$1" pin="VDD_IO"/>
 <wire x1="38.1" y1="127" x2="38.1" y2="132.08" width="0.1524" layer="91"/>
 <pinref part="C1" gate="G$1" pin="2"/>
@@
 <wire x1="22.86" y1="132.08" x2="15.24" y2="132.08" width="0.1524" layer="91"/>
 <pinref part="SUPPLY1" gate="G$1" pin="3.3V"/>
+<junction x="22.86" y="132.08"/>
 </segment>
 <segment>
-<pinref part="AKC+GYRO" gate="G$1" pin="!CS_A"/>
-<pinref part="AKC+GYRO" gate="G$1" pin="!CS_G"/>
+<pinref part="ACC+GYRO" gate="G$1" pin="!CS_A"/>
+<pinref part="ACC+GYRO" gate="G$1" pin="!CS_G"/>
 <wire x1="38.1" y1="172.72" x2="38.1" y2="177.8" width="0.1524" layer="91"/>
 <wire x1="38.1" y1="177.8" x2="20.32" y2="177.8" width="0.1524" layer="91"/>
@@
 <net name="SCL" class="0">
 <segment>
-<pinref part="AKC+GYRO" gate="G$1" pin="SCL"/>
+<pinref part="ACC+GYRO" gate="G$1" pin="SCL"/>
 <wire x1="38.1" y1="167.64" x2="30.48" y2="167.64" width="0.1524" layer="91"/>
 <label x="25.4" y="167.64" size="1.778" layer="95"/>
@@
 <net name="SDA" class="0">
 <segment>
-<pinref part="AKC+GYRO" gate="G$1" pin="SDA"/>
+<pinref part="ACC+GYRO" gate="G$1" pin="SDA"/>
 <wire x1="38.1" y1="152.4" x2="30.48" y2="152.4" width="0.1524" layer="91"/>
 <label x="25.4" y="152.4" size="1.778" layer="95"/>
 </segment>
 </net>
+<net name="INT_ACC" class="0">
+<segment>
+<pinref part="ACC+GYRO" gate="G$1" pin="INT1_A"/>
+<wire x1="81.28" y1="172.72" x2="86.36" y2="172.72" width="0.1524" layer="91"/>
+<label x="86.36" y="172.72" size="1.778" layer="95"/>
+</segment>
+</net>
+<net name="INT_GYRO" class="0">
+<segment>
+<pinref part="ACC+GYRO" gate="G$1" pin="INT1_G"/>
+<wire x1="81.28" y1="152.4" x2="86.36" y2="152.4" width="0.1524" layer="91"/>
+<label x="86.36" y="152.4" size="1.778" layer="95"/>
+</segment>
+</net>

Commit message: wartosci w lsm i schemat zigbee
Parts:
- C1: value (none) -> 100n
- C2: value (none) -> 10n
- C3: value (none) -> 10u
Changed lines of the file:
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@@
 <parts>
 <part name="ACC+GYRO" library="sensors-akc_zyr" deviceset="LSM330DLC" device=""/>
-<part name="C1" library="resistor" deviceset="C-EU" device="C0805"/>
-<part name="C2" library="resistor" deviceset="C-EU" device="C0805"/>
+<part name="C1" library="resistor" deviceset="C-EU" device="C0805" value="100n"/>
+<part name="C2" library="resistor" deviceset="C-EU" device="C0805" value="10n"/>
 <part name="GND1" library="supply1" deviceset="GND" device=""/>
 <part name="GND2" library="supply1" deviceset="GND" device=""/>
-<part name="C3" library="rcl" deviceset="CPOL-EU" device="SMCA"/>
+<part name="C3" library="rcl" deviceset="CPOL-EU" device="SMCA" value="10u"/>
 <part name="SUPPLY1" library="SparkFun-Aesthetics" deviceset="3.3V" device=""/>
 <part name="SUPPLY2" library="SparkFun-Aesthetics" deviceset="3.3V" device=""/>
